Commit message: 240612

File: my_env/Mag_Env/ur10e/ur10e.urdf (robot description, URDF)
Before this commit: robot ur10e, 8 links, 7 joints
Links:
- link base_link: geometry collision mesh filename=package://ur10e/collision/base.stl; visual mesh filename=package://ur10e/visual/base.dae
- link forearm_link: geometry collision mesh filename=package://ur10e/collision/forearm.stl; visual mesh filename=package://ur10e/visual/forearm.dae
- link ma: geometry collision mesh filename=package://ur10e/ma/meshes/ma2.STL; visual mesh filename=package://ur10e/ma/meshes/ma2.STL
- link shoulder_link: geometry collision mesh filename=package://ur10e/collision/shoulder.stl; visual mesh filename=package://ur10e/visual/shoulder.dae
- link upper_arm_link: geometry collision mesh filename=package://ur10e/collision/upperarm.stl; visual mesh filename=package://ur10e/visual/upperarm.dae
- link wrist_1_link: geometry collision mesh filename=package://ur10e/collision/wrist1.stl; visual mesh filename=package://ur10e/visual/wrist1.dae
- link wrist_2_link: geometry collision mesh filename=package://ur10e/collision/wrist2.stl; visual mesh filename=package://ur10e/visual/wrist2.dae
- link wrist_3_link: geometry collision mesh filename=package://ur10e/collision/wrist3.stl; visual mesh filename=package://ur10e/visual/wrist3.dae
Joints:
- joint tool0_fixed_joint: origin xyz=0 0.137 0 rpy=0 3.141592653589793 0 -> xyz=0 0.137 0 rpy=0 1.5707963267948966 0

Commit message: 20240711

File: my_env/Mag_Env/ur10e/ur10e.urdf (robot description, URDF)
Before this commit: robot ur10e, 8 links, 7 joints
Links:
- link base_link: geometry collision mesh filename=package://ur10e/collision/base.obj; visual mesh filename=package://ur10e/visual/base.dae
- link forearm_link: geometry collision mesh filename=package://ur10e/collision/forearm.obj; visual mesh filename=package://ur10e/visual/forearm.dae
- link ma: geometry collision mesh filename=package://ur10e/ma/meshes/ma.obj; visual mesh filename=package://ur10e/ma/meshes/ma.dae
- link shoulder_link: geometry collision mesh filename=package://ur10e/collision/shoulder.obj; visual mesh filename=package://ur10e/visual/shoulder.dae
- link upper_arm_link: geometry collision mesh filename=package://ur10e/collision/upperarm.obj; visual mesh filename=package://ur10e/visual/upperarm.dae
- link wrist_1_link: geometry collision mesh filename=package://ur10e/collision/wrist1.obj; visual mesh filename=package://ur10e/visual/wrist1.dae
- link wrist_2_link: geometry collision mesh filename=package://ur10e/collision/wrist2.obj; visual mesh filename=package://ur10e/visual/wrist2.dae
- link wrist_3_link: geometry collision mesh filename=package://ur10e/collision/wrist3.obj; visual mesh filename=package://ur10e/visual/wrist3.dae
